File: V2 KiCad Files/RP2040 Board.kicad_pcb (KiCad board)
At the start: 2 copper layers, 60 x 42 mm, 39 parts, among them J1 USB_C_Receptacle_USB2.0, SW1 USB Boot Button, SW2 Push_Button, SW3 Push_Button, SW4 Push_Button, SW5 Push_Button, SW6 Push_Button, U1 RP2040, U2 ADP3338AKCZ-3.3, U3 W25Q128JVSIQ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

Commit message: Add files via upload
Parts:
- removed R10, R11, R7, R8, R9: 1K, 1K Resistor:RC0402N_PAN
- removed R6: Resistor, Resistor_SMD:R_0201_0603Metric
- removed SW1: USB Boot Button, Push Button:SW4_1825910-B_TEC
- removed U2: ADP3338AKCZ-3.3, PCM_4ms_Package_SOT:SOT89-3
- added R5: 1K, 1K Resistor:RC0402N_PAN, B.Cu at (144.0, 72.5)
- added U4: NCP51460SN33, Voltage:NCP1117, F.Cu at (150.0, 78.0)
- C1, C10, C14_100n1, C2, C3, C4, C5, C6, C7, C9: value Capacitor_NP -> 100nF
- C11, C8: value Capacitor_NP -> 1uF
- C12: value Capacitor_NP -> 10uF
- C13: value Capacitor_NP -> 10uF; moved to B.Cu
- C14: value Capacitor 15pF -> 15pF
- J2: renamed from Test Pins
- R1, R2: value Resistor -> 27Ω
- moved C13 6.54 mm to (146.0, 79.0)
Connections:
- SW2 pad 2: Net-(R7-Pad2) -> GND
- SW3 pad 2: Net-(R8-Pad2) -> GND
- SW4 pad 2: Net-(R9-Pad2) -> GND
- SW5 pad 2: Net-(R10-Pad2) -> GND
- SW6 pad 2: Net-(R11-Pad2) -> GND
Routing:
- net 3v3: track 194.4 -> 128.3 mm, vias 13 -> 10
- net Net-(R6-Pad1): track 29.6 -> 0.00 mm
- net GND: track 12.1 -> 26.2 mm, vias 7 -> 11
- net GPIO22: track 53.9 -> 40.4 mm
- net RUN: track 59.2 -> 46.6 mm
- net GPIO11: track 16.1 -> 24.7 mm
- net GPIO21: track 30.3 -> 22.5 mm
- net (no net): track 6.99 -> 0.01 mm, vias 1 -> 0
- net unconnected-(U1-GND-Pad57): track 3.11 -> 7.38 mm
- net Net-(R9-Pad2): track 2.47 -> 0.00 mm
- net Net-(R7-Pad2): track 2.47 -> 0.00 mm
- net Net-(R10-Pad2): track 2.47 -> 0.00 mm
- net Net-(R11-Pad2): track 2.45 -> 0.00 mm
- net Net-(R8-Pad2): track 2.39 -> 0.00 mm
- net GPIO13: track 59.6 -> 58.2 mm

Commit message: Add files via upload
Parts:
- R1, R2, R3, R4: footprint Resistor_SMD:R_0201_0603Metric -> PCM_Resistor_SMD_AKL:R_0402_1005Metric
- U4: value NCP51460SN33 -> NCP1117LPST33T3G
- moved R2 0.60 mm to (137.5, 73.0)
- moved C11 0.50 mm to (137.5, 77.8)
- moved C14_100n1 0.50 mm to (136.2, 64.5)
- moved C5 0.50 mm to (144.2, 76.0)
- moved C8 0.50 mm to (130.2, 72.5)
- moved R3 0.50 mm to (150.2, 68.5)
- moved R4 0.50 mm to (147.2, 68.5)
- moved R1 0.34 mm to (139.0, 73.0)
Routing:
- net GND: track 26.2 -> 52.9 mm, vias 11 -> 12
- net unconnected-(U1-GND-Pad57): track 7.38 -> 0.00 mm
- net 3v3: track 128.3 -> 131.9 mm
- net GPIO13: track 58.2 -> 57.0 mm
- net GPIO21: track 22.5 -> 21.7 mm
- net Net-(J1-CC1): track 1.90 -> 2.48 mm
- net Net-(J1-CC2): track 1.84 -> 2.40 mm
- net GPIO11: track 24.7 -> 24.2 mm
- net Net-(U1-USB_DP): track 1.91 -> 1.37 mm
