File: V2 KiCad Files/RP2040 Board.kicad_sch (KiCad schematic)
At the start: 39 parts, among them J1 USB_C_Receptacle_USB2.0, J2 Test Pins, SW1 USB Boot Button, SW2 Push_Button, SW3 Push_Button, SW4 Push_Button, SW5 Push_Button, SW6 Push_Button, U1 RP2040, U2 ADP3338AKCZ-3.3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

Commit message: Add files via upload
Parts:
- removed R10, R11, R7, R8, R9: 1K, 1K Resistor:RC0402N_PAN, symbol ERJ-2RKF1001X 1k Resistor:ERJ-2RKF1001X
- removed R6: Resistor, Resistor_SMD:R_0201_0603Metric, symbol PCM_SL_Resistors:Resistor
- removed SW1: USB Boot Button, Push Button:SW4_1825910-B_TEC, symbol PCM_SL_Devices:Push_Button_W12mm
- removed U2: ADP3338AKCZ-3.3, PCM_4ms_Package_SOT:SOT89-3, symbol PCM_Voltage_Regulator_AKL:ADP3338AKCZ-3.3
- added R5: 1K, 1K Resistor:RC0402N_PAN, symbol ERJ-2RKF1001X 1k Resistor:ERJ-2RKF1001X
- added U4: NCP51460SN33, Voltage:NCP1117, symbol PCM_4ms_Reference:NCP51460SN33
- C1, C10, C14_100n1, C2, C3, C4, C5, C6, C7, C9: value Capacitor_NP -> 100nF; Manufacturer (none) -> Samsung Electro-Mechanics; Part Number (none) -> CL10E104KC8VPNC
- C11, C8: value Capacitor_NP -> 1uF
- C12, C13: value Capacitor_NP -> 10uF
- C14: value Capacitor 15pF -> 15pF
- R1, R2: value Resistor -> 27Ω
- X1: Manufacturer (none) -> Abracon LLC; Part Number (none) -> ABM8-272-T3
Connections:
- net 3v3: now also U4.2 (VO)
- net GND: now also SW2.2, SW3.2, SW4.2, SW5.2, SW6.2, U4.3 (GND)
- net GPIO11: now also R5.2
- net at U1.56 (QSPI_SS), U3.1 (/CS): now also R5.1
- net at C12.1, J1.A4 (VBUS), J1.A9 (VBUS)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: now also U4.1 (VI)
Other:
- note added: "Row 1"
- note added: "Row 2"
- moved on the sheet: SW2, SW3, SW4, SW5, SW6

Commit message: Add files via upload
Parts:
- C11, C8: Manufacturer (none) -> Samsung Electro-Mechanics; Part Number (none) -> CL10B105KP8NNNC
- C12, C13: Manufacturer (none) -> Samsung Electro-Mechanics; Part Number (none) -> CL10A106MQ8NNNC
- C14, C15: Manufacturer (none) -> Würth Elektronik; Part Number (none) -> 885012006003
- J1: Manufacturer (none) -> G-Switch; Part Number (none) -> GT-USB-7010ASV
- J2: footprint Connector_PinHeader_1.00mm:PinHeader_2x22_P1.00mm_Vertical -> (none)
- R1, R2: footprint Resistor_SMD:R_0201_0603Metric -> PCM_Resistor_SMD_AKL:R_0402_1005Metric; Manufacturer (none) -> Panasonic Electronic Components; Part Number (none) -> ERJ-2RKF27R0X
- R12, R5: Manufacturer (none) -> Panasonic Electronic Components; Part Number (none) -> ERJ-2RKF1001X
- R3, R4: footprint Resistor_SMD:R_0201_0603Metric -> PCM_Resistor_SMD_AKL:R_0402_1005Metric; Manufacturer (none) -> Panasonic Electronic Components; Part Number (none) -> ERA-2AEB512X
- SW2, SW3, SW4, SW5, SW6: Manufacturer (none) -> Cherry Americas LLC; Part Number (none) -> MX1A-C1NW
- U1: Manufacturer (none) -> Raspberry Pi; Part Number (none) -> SC0914(13)
- U3: Manufacturer (none) -> Winbond Electronics; Part Number (none) -> W25Q128JVSIQ
- U4: value NCP51460SN33 -> NCP1117LPST33T3G; Manufacturer ON Semiconductor -> onsemi; Part Number NCP51460SN33T1G -> NCP1117LPST33T3G
- X1: Manufacturer Abracon LLC -> Abracon LLC
